File: PCB/PrivaSee_V02/PrivaSee_V02.kicad_sch (KiCad schematic)
At the start: 33 parts, among them J1 RFPC-SMA27-F, J2 Batt_Solder_Point, J3 Conn_02x06_Odd_Even, J4 VOUT_TEST, J5 GND_TEST, J6 IR_TEST, J7 RF_TEST, SW1 Switch, SW2 SW_Push, U1 RC1602A, U2 LM358, U3 254, U4 DFR0568, U5 ESP32-C6-DevKitC-1

Commit message: Cleaning up some of the schematic
Discovered error in both the op amp placement and diode placement. New PCB order needed.
Parts:
- removed D1: BAT1504WH6327XTSA1, JLCImport:BAT1504WH6327XTSA1, symbol JLCImport:BAT1504WH6327XTSA1
- removed R2: 470 Ohm, Resistor_SMD:R_1206_3216Metric_Pad1.30x1.75mm_HandSolder, symbol Device:R_US
- added D2, D4: BAT_15-02EL_E6327, JLCImport:BAT_15-02EL_E6327, symbol JLCImport:BAT_15-02EL_E6327
Connections:
- net GND: now also C3.1, R6.2, D4.2 (A); no longer C3.2, R6.1
- net at J7.1 (Pin_1), U5.7 (GPIO0): now also R1.1, U2.1
- net at R1.2: now also R7.1, U2.2 (-); no longer U2.1
- net at C2.1: now also D2.2 (A), D4.1 (C)
- new net: C3.2, D2.1 (C), R6.1, U2.3 (+)
Other:
- moved on the sheet: R1, R7, Reference: C1, Reference: C2, Reference: C3, Reference: J1, Reference: L1, Reference: R6, U2A
